File: hardware/OpenTaxus.kicad_sch (KiCad schematic)
At the start: 56 parts, among them J1 OLED, J2 qwiic, J3 SWD, J4 USB_C_Receptacle_USB2.0, J5 connector, Q2 BC847BS, Q3 PT12-21B/TR8, SW1 dpad, SW2 USB_BOOT, SW3 RESET, SW4 SW_SPDT, SW5 USB_BOOT, U1 HE6206-33NR, U2 W25Q128JVS, U3 RP2040, U4 XT1861B332MR-G, Y1 YSX321SL

Commit message: De-branded the kicad files
Other:
- title: BSidesSF 2024 Badge -> OpenTaxus Badge
Changed lines of the file:
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@@
 	(paper "A4")
 	(title_block
-		(title "BSidesSF 2024 Badge")
-		(date "2024-03-06")
+		(title "OpenTaxus Badge")
+		(date "2024-06-12")
 		(rev "1.0")
 		(comment 1 "Joe FitzPatrick")
