File: hardware/OpenTaxus.kicad_pcb (KiCad board)
At the start: 2 copper layers, 66.7 x 85.7 mm, 55 parts, among them J1 OLED, J2 qwiic, J3 SWD, J4 USB_C_Receptacle_USB2.0, Q2 BC847BS, Q3 PT12-21B/TR8, SW1 dpad, SW2 USB_BOOT, SW3 RESET, SW4 SW_SPDT, U1 HE6206-33NR, U2 W25Q128JVS, U3 RP2040, U4 XT1861B332MR-G, Y1 YSX321SL

Commit message: Removed OH logo for licensing clarity
Parts:
- removed OSHW: OSHW-Logo2_14.6x12mm_SolderMask, logos:OSHW-Logo2_14.6x12mm_SolderMask
